File: esp_addressable_leds/esp-c3-addressable-leds.kicad_pcb (KiCad board)
At the start: 2 copper layers, 75 x 50 mm, 7 parts, among them J1 Conn_01x03, U2 74AHCT1G125

Commit message: add build script
Parts:
- added REF**: MountingHole_3.2mm_M3, MountingHole:MountingHole_3.2mm_M3, F.Cu at (111.0, 64.6)
- added REF**: MountingHole_3.2mm_M3, MountingHole:MountingHole_3.2mm_M3, F.Cu at (176.0, 104.6)

Commit message: update
Parts:
- removed REF** (x2): MountingHole_3.2mm_M3, MountingHole:MountingHole_3.2mm_M3
- added H1: MountingHole, MountingHole:MountingHole_3.2mm_M3, F.Cu at (110.5, 64.1)
- added H2: MountingHole, MountingHole:MountingHole_3.2mm_M3, F.Cu at (161.5, 105.1)
- J1: footprint Connector_Wire:SolderWire-0.5sqmm_1x03_P4.8mm_D0.9mm_OD2.3mm_Relief2x -> Connector_Wire:SolderWire-0.5sqmm_1x03_P4.8mm_D0.9mm_OD2.3mm_Relief
Other:
- board size 75 x 50 mm -> 60 x 50 mm
- board text added: "flaviutamas.com/p/esp-addressable-led"
