File: esp_cc_dimmer/esp_cc_dimmer.kicad_pcb (KiCad board)
At the start: 2 copper layers, 68.2 x 52 mm, 14 parts, among them J1 Conn_01x02, J2 Conn_01x02, SW1 RotaryEncoder_Switch, U2 VEML7700-TR, U3 XIAO-ESP32-C3-SMD

Commit message: done maybe
Parts:
- added REF**: MountingHole_3.2mm_M3, MountingHole:MountingHole_3.2mm_M3, F.Cu at (70.5, 117.2)
- added REF**: MountingHole_3.2mm_M3, MountingHole:MountingHole_3.2mm_M3, F.Cu at (70.5, 73.2)
Connections:
- SW1 pad MP: (no net) -> GND
Routing:
- net Net-(U3-GPIO4_A2_D2): track 51.5 -> 54.2 mm
- net Net-(U3-GPIO3_A1_D1): track 52.7 -> 55.3 mm
- net GND: vias 5 -> 6

Commit message: update
Parts:
- removed C10, C9: 10u, Capacitor_SMD:C_0805_2012Metric
- removed REF** (x2): MountingHole_3.2mm_M3, MountingHole:MountingHole_3.2mm_M3
- added C11: 4.7u 100V, Capacitor_SMD:C_1210_3225Metric_Pad1.33x2.70mm_HandSolder, F.Cu at (81.0, 86.0)
- added C2: 100u 63V, Capacitor_THT:CP_Radial_D8.0mm_P3.50mm, F.Cu at (74.3, 83.0)
- added H1: MountingHole, MountingHole:MountingHole_3.2mm_M3, F.Cu at (70.5, 73.2)
- added H2: MountingHole, MountingHole:MountingHole_3.2mm_M3, F.Cu at (70.5, 117.2)
- J1, J2: value Conn_01x02 -> WJ15EDGRC-3.81-02P-14-00A
- SW1: value RotaryEncoder_Switch -> EC11E15244G1
Routing:
- net +48V: track 30.7 -> 3.94 mm
- net +3V3: track 90.6 -> 105.5 mm, vias 2 -> 0
- net Net-(C10-Pad2): track 1.60 -> 0.00 mm
- net GND: track 15.1 -> 16.4 mm
- added copper zone on F.Cu, net +48V
Other:
- board text added: "48V"
- board text added: "GND"
- board text added: "LED+"
- board text added: "LED-"
- board text added: "flaviutamas.com/p/esp-cc-dimmer"

Commit message: fix bugs, add esphome config
Parts:
- C3: value 1u -> 1uF
- C8: footprint Capacitor_SMD:C_0805_2012Metric -> Capacitor_SMD:C_1210_3225Metric_Pad1.33x2.70mm_HandSolder
- U4: value ~ -> LX8015
- moved J2 1.60 mm to (74.3, 92.7)
- moved J1 0.40 mm to (127.0, 96.3)
- moved C8 0.20 mm to (105.9, 85.5)
Routing:
- net +5V: track 4.65 -> 0.00 mm
- net +48V: track 3.94 -> 0.00 mm
Changed lines of the file:
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@@
 			)
 		)
-		(property "Value" "~"
+		(property "Value" "LX8015"
 			(at 0 1 0)
 			(unlocked yes)
@@
 		(sheetname "/")
 		(sheetfile "esp_cc_dimmer.kicad_sch")
-		(units
-			(unit
-				(name "A")
-				(pins "1" "2" "3" "4")
-			)
-		)
 		(attr smd)
 		(duplicate_pad_numbers_are_jumpers no)
@@
 			)
 		)
-		(pad "1" thru_hole circle
-			(at -12.05 -6.3)
-			(size 2.4 2.4)
-			(drill 1.8)
+		(pad "1" thru_hole oval
+			(at -11 -6.25)
+			(size 3.8 2.6)
+			(drill oval 3 1.8)
 			(layers "*.Cu" "*.Mask")
 			(remove_unused_layers no)
@@
 			(pintype "power_in")
 		)
-		(pad "2" thru_hole circle
-			(at -12.05 6.3)
-			(size 2.4 2.4)
-			(drill 1.8)
+		(pad "2" thru_hole oval
+			(at -11.05 6.3)
+			(size 3.8 2.6)
+			(drill oval 3 1.8)
 			(layers "*.Cu" "*.Mask")
 			(remove_unused_layers no)
@@
 			(pintype "power_in")
 		)
-		(pad "3" thru_hole circle
-			(at 12.05 6.3)
-			(size 2.4 2.4)
-			(drill 1.8)
+		(pad "3" thru_hole oval
+			(at 11.05 6.3)
+			(size 3.8 2.6)
+			(drill oval 3 1.8)
 			(layers "*.Cu" "*.Mask")
 			(remove_unused_layers no)
@@
 			(pintype "power_in")
 		)
-		(pad "4" thru_hole circle
-			(at 12.05 -6.3)
-			(size 2.4 2.4)
-			(drill 1.8)
+		(pad "4" thru_hole oval
+			(at 11.05 -6.3)
+			(size 3.8 2.6)
+			(drill oval 3 1.8)
 			(layers "*.Cu" "*.Mask")
 			(remove_unused_layers no)
@@
 		(embedded_fonts no)
 	)
-	(footprint "Capacitor_SMD:C_0805_2012Metric"
+	(footprint "Capacitor_SMD:C_1210_3225Metric_Pad1.33x2.70mm_HandSolder"
 		(layer "F.Cu")
-		(at 105.7 85.45 -90)
-		(descr "Capacitor SMD 0805 (2012 Metric), square (rectangular) end terminal, IPC-7351 nominal, (Body size source: IPC-SM-782 page 76, https://www.pcb-3d.com/wordpress/wp-content/uploads/ipc-sm-782a_amendment_1_and_2.pdf, https://docs.google.com/spreadsheets/d/1BsfQQcO9C6DZCsRaXUlFlo91Tg2WpOkGARC1WS5S8t0/edit?usp=sharing)")
-		(tags "capacitor")
+		(at 105.9 85.45 -90)
+		(descr "Capacitor SMD 1210 (3225 Metric), square (rectangular) end terminal, IPC-7351 nominal with elongated pad for handsoldering. (Body size source: IPC-SM-782 page 76, https://www.pcb-3d.com/wordpress/wp-content/uploads/ipc-sm-782a_amendment_1_and_2.pdf)")
+		(tags "capacitor handsolder")
 		(property "Reference" "C8"
-			(at 2.5 0 0)
+			(at 0 -2.3 270)
 			(layer "F.SilkS")
 			(effects
@@
 		)
 		(property "Value" "10u"
-			(at 0 1.68 90)
+			(at 0 2.3 270)
 			(layer "F.Fab")
 			(effects
@@
 		)
 		(property "Datasheet" ""
-			(at 0 0 90)
+			(at 0 0 270)
 			(layer "F.Fab")
 			(hide yes)
@@
 		)
 		(property "Description" "Unpolarized capacitor"
-			(at 0 0 90)
+			(at 0 0 270)
 			(layer "F.Fab")
 			(hide yes)
@@
 		)
 		(property "KiLib_Generator" "SMD_2terminal_chip_molded"
-			(at 0 0 90)
+			(at 0 0 270)
 			(layer "F.SilkS")
 			(hide yes)
@@
 		(duplicate_pad_numbers_are_jumpers no)
 		(fp_line
-			(start -0.261252 0.735)
-			(end 0.261252 0.735)
+			(start -0.711252 1.36)
+			(end 0.711252 1.36)
 			(stroke
 				(width 0.12)
@@
 		)
 		(fp_line
-			(start -0.261252 -0.735)
-			(end 0.261252 -0.735)
+			(start -0.711252 -1.36)
+			(end 0.711252 -1.36)
 			(stroke
 				(width 0.12)
@@
 		)
 		(fp_rect
-			(start -1.7 -0.98)
-			(end 1.7 0.98)
+			(start -2.48 -1.6)
+			(end 2.48 1.6)
 			(stroke
 				(width 0.05)
@@
 		)
 		(fp_rect
-			(start -1 -0.625)
-			(end 1 0.625)
+			(start -1.6 -1.25)
+			(end 1.6 1.25)
 			(stroke
 				(width 0.1)
@@
 		)
 		(fp_text user "${REFERENCE}"
-			(at 0 0 90)
+			(at 0 0 270)
 			(layer "F.Fab")
 			(effects
 				(font
-					(size 0.5 0.5)
-					(thickness 0.08)
+					(size 0.8 0.8)
+					(thickness 0.12)
 				)
 			)
 		)
 		(pad "1" smd roundrect
-			(at -0.95 0 270)
-			(size 1 1.45)
+			(at -1.5625 0 270)
+			(size 1.325 2.7)
 			(layers "F.Cu" "F.Mask" "F.Paste")
-			(roundrect_rratio 0.25)
+			(roundrect_rratio 0.188679)
 			(net "+5V")
 			(pintype "passive")
 		)
 		(pad "2" smd roundrect
-			(at 0.95 0 270)
-			(size 1 1.45)
+			(at 1.5625 0 270)
+			(size 1.325 2.7)
 			(layers "F.Cu" "F.Mask" "F.Paste")
-			(roundrect_rratio 0.25)
+			(roundrect_rratio 0.188679)
 			(net "GND")
 			(pintype "passive")
 		)
 		(embedded_fonts no)
-		(model "${KICAD10_3DMODEL_DIR}/Capacitor_SMD.3dshapes/C_0805_2012Metric.step"
+		(model "${KICAD10_3DMODEL_DIR}/Capacitor_SMD.3dshapes/C_1210_3225Metric.step"
 			(offset
 				(xyz 0 0 0)
@@
 			)
 		)
-		(property "Value" "1u"
+		(property "Value" "1uF"
 			(at 0 1.43 90)
 			(layer "F.Fab")
@@
 	(footprint "Connector_Phoenix_MC:PhoenixContact_MC_1,5_2-G-3.81_1x02_P3.81mm_Horizontal"
 		(layer "F.Cu")
-		(at 75.9325 92.65 -90)
+		(at 74.3325 92.65 -90)
 		(descr "Generic Phoenix Contact connector footprint for: MC_1,5/2-G-3.81; number of pins: 02; pin pitch: 3.81mm; Angled || order number: 1803277 8A 160V")
 		(tags "phoenix_contact connector MC_01x02_G_3.81mm")
@@
 	(footprint "Connector_Phoenix_MC:PhoenixContact_MC_1,5_2-G-3.81_1x02_P3.81mm_Horizontal"
 		(layer "F.Cu")
-		(at 126.5675 96.35 90)
+		(at 126.9675 96.35 90)
 		(descr "Generic Phoenix Contact connector footprint for: MC_1,5/2-G-3.81; number of pins: 02; pin pitch: 3.81mm; Angled || order number: 1803277 8A 160V")
 		(tags "phoenix_contact connector MC_01x02_G_3.81mm")
@@
 	)
 	(segment
+		(start 105.7 87.0125)
+		(end 105.7 92.15)
+		(width 0.6)
+		(layer "F.Cu")
+		(net "GND")
+	)
+	(segment
 		(start 120.45 99.95)
 		(end 120.5 100)
@@
 	)
 	(segment
-		(start 84.2 74.8)
-		(end 84.2 73.55)
-		(width 0.2)
+		(start 105.7 92.15)
+		(end 105.55 92.3)
+		(width 0.6)
 		(layer "F.Cu")
 		(net "GND")
 	)
 	(segment
-		(start 105.7 86.4)
-		(end 105.7 92.15)
-		(width 0.6)
+		(start 84.2 74.8)
+		(end 84.2 73.55)
+		(width 0.2)
 		(layer "F.Cu")
 		(net "GND")
@@
 	)
 	(segment
-		(start 82.01 99.495)
-		(end 82.01 98.7275)
-		(width 2)
-		(layer "F.Cu")
-		(net "+48V")
-	)
-	(segment
-		(start 81 80.15)
-		(end 81.45 79.7)
-		(width 1.2)
-		(layer "F.Cu")
-		(net "+48V")
-	)
-	(segment
-		(start 82.01 99.495)
-		(end 84.55 99.495)
-		(width 2)
-		(layer "F.Cu")
-		(net "+48V")
-	)
-	(segment
-		(start 105.7 84.5)
-		(end 105.7 79.85)
-		(width 0.6)
-		(layer "F.Cu")
-		(net "+5V")
-	)
-	(segment
 		(start 127.468 109.5)
 		(end 127.468 113.968)
@@
 	(group ""
 		(members "090a27e0-36e0-40b9-a648-18542ae0c39f" "0f2f02dd-9511-4b92-b232-dc644ad11506"
-			"1cb98002-2aa5-4692-adc7-a858a8fc2e9a" "82462b48-703c-4dd2-8120-f4d426b7c113"
-			"e8f34c76-7ed9-412b-90e4-e193342bd5bf" "fd080f72-d351-47c9-baed-e16bce14b7c7"
-			"fe7442bc-ec59-4794-bc3f-80bad15fd29e"
+			"1cb98002-2aa5-4692-adc7-a858a8fc2e9a" "2703b6c3-0bb3-4e37-ae6a-9e1395949049"
+			"82462b48-703c-4dd2-8120-f4d426b7c113" "bf409d89-b303-49a2-bc8b-3aa8ba807554"
+			"fd080f72-d351-47c9-baed-e16bce14b7c7"
 		)
 	)
